Commit message: 뒷바퀴 2륜 구동
Co-Authored-By: Claude Sonnet 4.6 <noreply@anthropic.com>

File: src/fw_mini_description/urdf/fw_mini.gazebo.xacro (robot description, xacro)
@@ -26,56 +26,23 @@
   </gazebo>
   <gazebo reference="left_front_wheel">
-    <mu1>1.0</mu1>
-    <mu2>2.0</mu2>
+    <mu1>0.5</mu1>
+    <mu2>0.0</mu2>
     <kp>10000000.0</kp>
     <kd>1.0</kd>
-    <fdir1>0 0 1</fdir1>
     <material>Gazebo/Black</material>
   </gazebo>
   <gazebo reference="right_front_wheel">
-    <mu1>1.0</mu1>
-    <mu2>2.0</mu2>
+    <mu1>0.5</mu1>
+    <mu2>0.0</mu2>
     <kp>10000000.0</kp>
     <kd>1.0</kd>
-    <fdir1>0 0 1</fdir1>
     <material>Gazebo/Black</material>
   </gazebo>
-  <!-- Differential drive plugin (cmd_vel → odom 직접 퍼블리시, Nav2 연결용) -->
+  <!-- gazebo_ros2_control: ros2_control 하드웨어 인터페이스 -->
   <gazebo>
-    <plugin name="diff_drive" filename="libgazebo_ros_diff_drive.so">
-      <ros>
-        <remapping>cmd_vel:=cmd_vel</remapping>
-        <remapping>odom:=odom</remapping>
-      </ros>
-      <!-- 후륜 2개를 구동 바퀴로 사용 -->
-      <left_joint>left_rear_wheel_joint</left_joint>
-      <right_joint>right_rear_wheel_joint</right_joint>
-      <!-- 로봇 치수 (바퀴 반지름: 0.07m, 좌우 바퀴 간격: 0.25m) -->
-      <wheel_separation>0.25</wheel_separation>
-      <wheel_diameter>0.14</wheel_diameter>
-      <max_wheel_torque>20</max_wheel_torque>
-      <max_wheel_acceleration>1.0</max_wheel_acceleration>
-      <publish_odom>true</publish_odom>
-      <publish_odom_tf>true</publish_odom_tf>
-      <publish_wheel_tf>false</publish_wheel_tf>
-      <odometry_frame>odom</odometry_frame>
-      <robot_base_frame>base_footprint</robot_base_frame>
-    </plugin>
-  </gazebo>
-  <!-- joint_state_publisher (wheel joint states 퍼블리시) -->
-  <gazebo>
-    <plugin name="joint_state_publisher" filename="libgazebo_ros_joint_state_publisher.so">
-      <ros>
-        <remapping>~/out:=joint_states</remapping>
-      </ros>
-      <update_rate>50</update_rate>
-      <joint_name>right_rear_wheel_joint</joint_name>
-      <joint_name>left_rear_wheel_joint</joint_name>
-      <joint_name>right_front_wheel_joint</joint_name>
-      <joint_name>left_front_wheel_joint</joint_name>
-      <joint_name>right_steering_hinge_joint</joint_name>
-      <joint_name>left_steering_hinge_joint</joint_name>
-      <joint_name>rear_right_steering_hinge_joint</joint_name>
-      <joint_name>rear_left_steering_hinge_joint</joint_name>
+    <plugin name="gazebo_ros2_control" filename="libgazebo_ros2_control.so">
+      <parameters>$(find fw_mini_description)/config/controllers.yaml</parameters>
+      <robot_param>robot_description</robot_param>
+      <robot_param_node>robot_state_publisher</robot_param_node>
     </plugin>
   </gazebo>

File: src/fw_mini_description/urdf/fw_mini.urdf.xacro (robot description, xacro)
@@ -75,10 +75,8 @@
     </inertial>
   </link>
-  <joint name="left_steering_hinge_joint" type="revolute">
+  <joint name="left_steering_hinge_joint" type="fixed">
     <parent link="base_link"/>
     <child link="left_steering_hinge"/>
     <origin xyz="0.175 0.125 0"/>
-    <axis xyz="0 0 1"/>
-    <limit lower="-1.57" upper="1.57" effort="10.0" velocity="50.0"/>
   </joint>
   <link name="left_front_wheel">
@@ -126,10 +124,8 @@
     </inertial>
   </link>
-  <joint name="right_steering_hinge_joint" type="revolute">
+  <joint name="right_steering_hinge_joint" type="fixed">
     <parent link="base_link"/>
     <child link="right_steering_hinge"/>
     <origin xyz="0.175 -0.125 0"/>
-    <axis xyz="0 0 1"/>
-    <limit lower="-1.57" upper="1.57" effort="10.0" velocity="50.0"/>
   </joint>
   <link name="right_front_wheel">
@@ -177,10 +173,8 @@
     </inertial>
   </link>
-  <joint name="rear_left_steering_hinge_joint" type="revolute">
+  <joint name="rear_left_steering_hinge_joint" type="fixed">
     <parent link="base_link"/>
     <child link="rear_left_steering_hinge"/>
     <origin xyz="-0.175 0.125 0"/>
-    <axis xyz="0 0 1"/>
-    <limit lower="-1.57" upper="1.57" effort="10.0" velocity="50.0"/>
   </joint>
   <link name="left_rear_wheel">
@@ -228,10 +222,8 @@
     </inertial>
   </link>
-  <joint name="rear_right_steering_hinge_joint" type="revolute">
+  <joint name="rear_right_steering_hinge_joint" type="fixed">
     <parent link="base_link"/>
     <child link="rear_right_steering_hinge"/>
     <origin xyz="-0.175 -0.125 0"/>
-    <axis xyz="0 0 1"/>
-    <limit lower="-1.57" upper="1.57" effort="10.0" velocity="50.0"/>
   </joint>
   <link name="right_rear_wheel">

File: src/fw_mini_description/urdf/macros.xacro (robot description, xacro)
@@ -1,5 +1,19 @@
 <?xml version="1.0"?>
 <robot name="fw_mini" xmlns:xacro="http://www.ros.org/wiki/xacro">
-  <!-- 현재 시뮬레이션은 gazebo_ros_diff_drive 플러그인으로 구동 -->
-  <!-- ros2_control 기반 컨트롤러가 필요할 때 여기에 추가 -->
+  <ros2_control name="fw_mini_hardware" type="system">
+    <hardware>
+      <plugin>gazebo_ros2_control/GazeboSystem</plugin>
+    </hardware>
+    <!-- 뒤 구동 바퀴 (velocity) -->
+    <joint name="left_rear_wheel_joint">
+      <command_interface name="velocity"/>
+      <state_interface name="velocity"/>
+      <state_interface name="position"/>
+    </joint>
+    <joint name="right_rear_wheel_joint">
+      <command_interface name="velocity"/>
+      <state_interface name="velocity"/>
+      <state_interface name="position"/>
+    </joint>
+  </ros2_control>
 </robot>

Commit message: 260327 퇴근전
Co-Authored-By: Claude Opus 4.6 (1M context) <noreply@anthropic.com>

File: src/fw_mini_description/urdf/fw_mini.gazebo.xacro (robot description, xacro)
@@ -3,6 +3,6 @@
   <!-- Gazebo material / friction properties -->
   <gazebo reference="base_link">
-    <mu1>0.0</mu1>
-    <mu2>0.0</mu2>
+    <mu1>1.0</mu1>
+    <mu2>0.9</mu2>
     <kp>10000000.0</kp>
     <kd>1.0</kd>
@@ -10,6 +10,6 @@
   </gazebo>
   <gazebo reference="left_rear_wheel">
-    <mu1>1.0</mu1>
-    <mu2>2.0</mu2>
+    <mu1>0.2</mu1>
+    <mu2>0.2</mu2>
     <kp>10000000.0</kp>
     <kd>1.0</kd>
@@ -18,6 +18,6 @@
   </gazebo>
   <gazebo reference="right_rear_wheel">
-    <mu1>1.0</mu1>
-    <mu2>2.0</mu2>
+    <mu1>0.2</mu1>
+    <mu2>0.2</mu2>
     <kp>10000000.0</kp>
     <kd>1.0</kd>
@@ -26,5 +26,5 @@
   </gazebo>
   <gazebo reference="left_front_wheel">
-    <mu1>0.1</mu1>
+    <mu1>0.2</mu1>
     <mu2>0.2</mu2>
     <kp>10000000.0</kp>
@@ -33,5 +33,5 @@
   </gazebo>
   <gazebo reference="right_front_wheel">
-    <mu1>0.1</mu1>
+    <mu1>0.2</mu1>
     <mu2>0.2</mu2>
     <kp>10000000.0</kp>
@@ -39,10 +39,24 @@
     <material>Gazebo/Black</material>
   </gazebo>
-  <!-- gazebo_ros2_control: ros2_control 하드웨어 인터페이스 -->
+  <!-- diff_drive plugin: 4륜 skid-steer -->
   <gazebo>
-    <plugin name="gazebo_ros2_control" filename="libgazebo_ros2_control.so">
-      <parameters>$(find fw_mini_description)/config/controllers.yaml</parameters>
-      <robot_param>robot_description</robot_param>
-      <robot_param_node>robot_state_publisher</robot_param_node>
+    <plugin name="skid_steer_drive" filename="libgazebo_ros_diff_drive.so">
+      <update_rate>50</update_rate>
+      <num_wheel_pairs>2</num_wheel_pairs>
+      <left_joint>left_rear_wheel_joint</left_joint>
+      <left_joint>left_front_wheel_joint</left_joint>
+      <right_joint>right_rear_wheel_joint</right_joint>
+      <right_joint>right_front_wheel_joint</right_joint>
+      <wheel_separation>0.25</wheel_separation>
+      <wheel_separation>0.25</wheel_separation>
+      <wheel_diameter>0.14</wheel_diameter>
+      <wheel_diameter>0.14</wheel_diameter>
+      <max_wheel_torque>200</max_wheel_torque>
+      <max_wheel_acceleration>10.0</max_wheel_acceleration>
+      <publish_odom>true</publish_odom>
+      <publish_odom_tf>true</publish_odom_tf>
+      <publish_wheel_tf>false</publish_wheel_tf>
+      <odometry_frame>odom</odometry_frame>
+      <robot_base_frame>base_footprint</robot_base_frame>
     </plugin>
   </gazebo>

File: src/fw_mini_description/urdf/fw_mini.urdf.xacro (robot description, xacro)
@@ -89,6 +89,6 @@
     </visual>
     <collision>
-      <geometry><cylinder radius="0.07" length="0.05"/></geometry>
-      <origin xyz="0 0 0" rpy="1.57 0 0"/>
+      <geometry><sphere radius="0.07"/></geometry>
+      <origin xyz="0 0 0"/>
     </collision>
     <inertial>
@@ -138,6 +138,6 @@
     </visual>
     <collision>
-      <geometry><cylinder radius="0.07" length="0.05"/></geometry>
-      <origin xyz="0 0 0" rpy="1.57 0 0"/>
+      <geometry><sphere radius="0.07"/></geometry>
+      <origin xyz="0 0 0"/>
     </collision>
     <inertial>
@@ -187,6 +187,6 @@
     </visual>
     <collision>
-      <geometry><cylinder radius="0.07" length="0.05"/></geometry>
-      <origin xyz="0 0 0" rpy="1.57 0 0"/>
+      <geometry><sphere radius="0.07"/></geometry>
+      <origin xyz="0 0 0"/>
     </collision>
     <inertial>
@@ -236,6 +236,6 @@
     </visual>
     <collision>
-      <geometry><cylinder radius="0.07" length="0.05"/></geometry>
-      <origin xyz="0 0 0" rpy="1.57 0 0"/>
+      <geometry><sphere radius="0.07"/></geometry>
+      <origin xyz="0 0 0"/>
     </collision>
     <inertial>

File: src/fw_mini_description/urdf/macros.xacro (robot description, xacro)
@@ -1,19 +1,3 @@
 <?xml version="1.0"?>
 <robot name="fw_mini" xmlns:xacro="http://www.ros.org/wiki/xacro">
-  <ros2_control name="fw_mini_hardware" type="system">
-    <hardware>
-      <plugin>gazebo_ros2_control/GazeboSystem</plugin>
-    </hardware>
-    <!-- 뒤 구동 바퀴 (velocity) -->
-    <joint name="left_rear_wheel_joint">
-      <command_interface name="velocity"/>
-      <state_interface name="velocity"/>
-      <state_interface name="position"/>
-    </joint>
-    <joint name="right_rear_wheel_joint">
-      <command_interface name="velocity"/>
-      <state_interface name="velocity"/>
-      <state_interface name="position"/>
-    </joint>
-  </ros2_control>
 </robot>
